File: pico-en-control.kicad/pico-en-control.kicad_pcb (KiCad board)
At the start: 2 copper layers, 21 x 33.8 mm, 18 parts, among them J1 JST-PH2 Bat, J2 Pico Pin 1-13, J3 Pico Pin 40-28, J4 Alt-Bat, SW1 SW_Push_SLIM, U1 SN74HC74N, U2 PCF8563T, Y1 Crystal

Commit message: Rev 3.1 (prod)
Parts:
- moved R1 1.60 mm to (115.3, 114.1), turned to 0 degrees
Connections:
- J2 pad 6: /GP4_CLKOUT -> /GP4_DONE
- J2 pad 7: /GP5_DONE -> /GP5_CLKOUT
- JP1 pad 1: /GP4_CLKOUT -> /GP5_CLKOUT
- R1 pad 2: /GP5_DONE -> /GP4_DONE
- U1 pad 3: /GP5_DONE -> /GP4_DONE
Routing:
- net /GP4_DONE: track 0.00 -> 17.9 mm, vias 0 -> 1
- net /GP5_DONE: track 13.2 -> 0.00 mm, vias 1 -> 0
- net /GP5_CLKOUT: track 0.00 -> 3.73 mm
- net /GP4_CLKOUT: track 2.27 -> 0.00 mm
Other:
- board text added: "1"
- board text added: "40"
- board text added: "C"
- board text added: "D"
- board text added: "GP4_DONE"
- board text added: "GP5_CLKOUT"
- board text added: "github.com/bablokb/pico-en-control Rev. 3.1"
- board text removed: "GP4_CLKOUT"
- board text removed: "GP5_DONE"
- board text removed: "github.com/bablokb/pico-en-control Rev. 3"
