File: pico-en-control.kicad/pico-en-control.kicad_sch (KiCad schematic)
At the start: 17 parts, among them J1 JST-PH2 Bat, J2 Pico Pin 1-13, J3 Pico Pin 40-28, SW1 SW_Push_SLIM, U1 SN74HC74N, U2 PCF8563T, Y1 Crystal

Commit message: Rev3
Parts:
- added J4: Alt-Bat, Connector_PinHeader_2.54mm:PinHeader_1x02_P2.54mm_Vertical, symbol Connector_Generic:Conn_01x02
Connections:
- net +BATT: now also J4.1 (Pin_1)
- net GND: now also J4.2 (Pin_2)
Other:
- moved on the sheet: J1
Changed lines of the file:
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@@
   (title_block
     (title "pico-en-control")
-    (date "2023-02-03")
-    (rev "2")
+    (date "2023-02-09")
+    (rev "3")
     (company "Bernhard Bablok")
     (comment 1 "https://github.com/bablokb/pcb-pico-en-control")
   )
+  (junction (at 168.91 104.14) (diameter 0) (color 0 0 0 0)
+  )
   (junction (at 188.595 46.99) (diameter 0) (color 0 0 0 0)
   )
@@
   )
   (junction (at 192.405 67.31) (diameter 0) (color 0 0 0 0)
+  )
+  (junction (at 166.37 106.68) (diameter 0) (color 0 0 0 0)
   )
   (no_connect (at 88.9 128.27))
@@
     (stroke (width 0) (type default) (color 0 0 0 0))
   )
+  (wire (pts (xy 166.37 106.68) (xy 166.37 115.57))
+    (stroke (width 0) (type default) (color 0 0 0 0))
+  )
   (wire (pts (xy 123.825 114.935) (xy 127.635 114.935))
     (stroke (width 0) (type default) (color 0 0 0 0))
   )
+  (wire (pts (xy 168.91 115.57) (xy 166.37 115.57))
+    (stroke (width 0) (type default) (color 0 0 0 0))
+  )
   (wire (pts (xy 194.31 69.85) (xy 188.595 69.85))
     (stroke (width 0) (type default) (color 0 0 0 0))
@@
     (stroke (width 0) (type default) (color 0 0 0 0))
   )
+  (wire (pts (xy 166.37 106.68) (xy 168.91 106.68))
+    (stroke (width 0) (type default) (color 0 0 0 0))
+  )
   (polyline (pts (xy 151.765 98.425) (xy 231.14 98.425))
     (stroke (width 0) (type default) (color 0 0 0 0))
@@
     (stroke (width 0) (type default) (color 0 0 0 0))
   )
-  (wire (pts (xy 165.1 113.03) (xy 168.91 113.03))
+  (wire (pts (xy 165.1 104.14) (xy 168.91 104.14))
     (stroke (width 0) (type default) (color 0 0 0 0))
   )
@@
     (stroke (width 0) (type default) (color 0 0 0 0))
   )
+  (wire (pts (xy 168.91 104.14) (xy 168.91 113.03))
+    (stroke (width 0) (type default) (color 0 0 0 0))
+  )
   (wire (pts (xy 192.405 74.93) (xy 192.405 67.31))
     (stroke (width 0) (type default) (color 0 0 0 0))
@@
     (stroke (width 0) (type default) (color 0 0 0 0))
   )
-  (wire (pts (xy 165.1 115.57) (xy 168.91 115.57))
+  (wire (pts (xy 165.1 106.68) (xy 166.37 106.68))
     (stroke (width 0) (type default) (color 0 0 0 0))
   )
@@
     (pin "2")
   )
-  (symbol (lib_id "Connector_Generic:Conn_01x02") (at 173.99 113.03 0) (unit 1)
-    (in_bom yes) (on_board yes) (fields_autoplaced)
-    (property "Reference" "J1" (id 0) (at 176.022 113.4653 0)
-      (effects (font (size 1.27 1.27)) (justify left))
-    )
-    (property "Value" "JST-PH2 Bat" (id 1) (at 176.022 116.0022 0)
-      (effects (font (size 1.27 1.27)) (justify left))
-    )
-    (property "Footprint" "Connector_JST:JST_PH_S2B-PH-SM4-TB_1x02-1MP_P2.00mm_Horizontal" (id 2) (at 173.99 113.03 0)
-      (effects (font (size 1.27 1.27)) hide)
-    )
-    (property "Datasheet" "~" (id 3) (at 173.99 113.03 0)
+  (symbol (lib_id "Connector_Generic:Conn_01x02") (at 173.99 104.14 0) (unit 1)
+    (in_bom yes) (on_board yes) (fields_autoplaced)
+    (property "Reference" "J1" (id 0) (at 176.022 104.5753 0)
+      (effects (font (size 1.27 1.27)) (justify left))
+    )
+    (property "Value" "JST-PH2 Bat" (id 1) (at 176.022 107.1122 0)
+      (effects (font (size 1.27 1.27)) (justify left))
+    )
+    (property "Footprint" "Connector_JST:JST_PH_S2B-PH-SM4-TB_1x02-1MP_P2.00mm_Horizontal" (id 2) (at 173.99 104.14 0)
+      (effects (font (size 1.27 1.27)) hide)
+    )
+    (property "Datasheet" "~" (id 3) (at 173.99 104.14 0)
       (effects (font (size 1.27 1.27)) hide)
     )
@@
     (pin "2")
   )
-  (symbol (lib_id "power:GND") (at 165.1 115.57 270) (unit 1)
-    (in_bom yes) (on_board yes)
-    (property "Reference" "#PWR013" (id 0) (at 158.75 115.57 0)
-      (effects (font (size 1.27 1.27)) hide)
-    )
-    (property "Value" "GND" (id 1) (at 156.845 115.57 90)
-      (effects (font (size 1.27 1.27)) (justify left))
-    )
-    (property "Footprint" "" (id 2) (at 165.1 115.57 0)
-      (effects (font (size 1.27 1.27)) hide)
-    )
-    (property "Datasheet" "" (id 3) (at 165.1 115.57 0)
+  (symbol (lib_id "power:GND") (at 165.1 106.68 270) (unit 1)
+    (in_bom yes) (on_board yes)
+    (property "Reference" "#PWR013" (id 0) (at 158.75 106.68 0)
+      (effects (font (size 1.27 1.27)) hide)
+    )
+    (property "Value" "GND" (id 1) (at 156.845 106.68 90)
+      (effects (font (size 1.27 1.27)) (justify left))
+    )
+    (property "Footprint" "" (id 2) (at 165.1 106.68 0)
+      (effects (font (size 1.27 1.27)) hide)
+    )
+    (property "Datasheet" "" (id 3) (at 165.1 106.68 0)
       (effects (font (size 1.27 1.27)) hide)
     )
@@
     )
     (pin "1")
+  )
+  (symbol (lib_id "Connector_Generic:Conn_01x02") (at 173.99 113.03 0) (unit 1)
+    (in_bom yes) (on_board yes) (fields_autoplaced)
+    (property "Reference" "J4" (id 0) (at 176.022 113.4653 0)
+      (effects (font (size 1.27 1.27)) (justify left))
+    )
+    (property "Value" "Alt-Bat" (id 1) (at 176.022 116.0022 0)
+      (effects (font (size 1.27 1.27)) (justify left))
+    )
+    (property "Footprint" "Connector_PinHeader_2.54mm:PinHeader_1x02_P2.54mm_Vertical" (id 2) (at 173.99 113.03 0)
+      (effects (font (size 1.27 1.27)) hide)
+    )
+    (property "Datasheet" "~" (id 3) (at 173.99 113.03 0)
+      (effects (font (size 1.27 1.27)) hide)
+    )
+    (pin "1")
+    (pin "2")
   )
   (symbol (lib_id "power:GND") (at 201.295 76.835 0) (unit 1)
@@
     (pin "1")
   )
-  (symbol (lib_id "power:+BATT") (at 165.1 113.03 90) (unit 1)
-    (in_bom yes) (on_board yes) (fields_autoplaced)
-    (property "Reference" "#PWR012" (id 0) (at 168.91 113.03 0)
-      (effects (font (size 1.27 1.27)) hide)
-    )
-    (property "Value" "+BATT" (id 1) (at 161.925 113.4638 90)
-      (effects (font (size 1.27 1.27)) (justify left))
-    )
-    (property "Footprint" "" (id 2) (at 165.1 113.03 0)
-      (effects (font (size 1.27 1.27)) hide)
-    )
-    (property "Datasheet" "" (id 3) (at 165.1 113.03 0)
+  (symbol (lib_id "power:+BATT") (at 165.1 104.14 90) (unit 1)
+    (in_bom yes) (on_board yes) (fields_autoplaced)
+    (property "Reference" "#PWR012" (id 0) (at 168.91 104.14 0)
+      (effects (font (size 1.27 1.27)) hide)
+    )
+    (property "Value" "+BATT" (id 1) (at 161.925 104.5738 90)
+      (effects (font (size 1.27 1.27)) (justify left))
+    )
+    (property "Footprint" "" (id 2) (at 165.1 104.14 0)
+      (effects (font (size 1.27 1.27)) hide)
+    )
+    (property "Datasheet" "" (id 3) (at 165.1 104.14 0)
       (effects (font (size 1.27 1.27)) hide)
     )
@@
       (reference "J3") (unit 1) (value "Pico Pin 40-28") (footprint "user:Connector_1x13_no_solder")
     )
+    (path "/7a4f6e16-8d7b-416b-9aae-02528b9b9a08"
+      (reference "J4") (unit 1) (value "Alt-Bat") (footprint "Connector_PinHeader_2.54mm:PinHeader_1x02_P2.54mm_Vertical")
+    )
     (path "/668b2fa7-ee2a-4acf-9d0b-11a6a168259d"

Commit message: Rev 3.1 (prod)
Parts:
- J1, J2, J3, J4, SW1: now left out of the parts list
Connections:
- net GP4_CLKOUT renamed GP4_DONE
- net GP4_DONE: now also R1.2, U1.3 (1CLK); no longer JP1.1 (A)
- removed net GP5_DONE: J2.7 (Pin_7), R1.2, U1.3 (1CLK)
- new net GP5_CLKOUT: J2.7 (Pin_7), JP1.1 (A)
Changed lines of the file:
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@@
   (title_block
     (title "pico-en-control")
-    (date "2023-02-09")
-    (rev "3")
+    (date "2023-02-17")
+    (rev "3.1")
     (company "Bernhard Bablok")
     (comment 1 "https://github.com/bablokb/pcb-pico-en-control")
@@
     (effects (font (size 1.27 1.27)) (justify left bottom))
   )
-  (label "GP5_DONE" (at 127.635 122.555 0)
+  (label "GP5_CLKOUT" (at 127.635 122.555 0)
     (effects (font (size 1.27 1.27)) (justify left bottom))
   )
@@
     (effects (font (size 1.27 1.27)) (justify left bottom))
   )
-  (label "GP4_CLKOUT" (at 127 90.17 0)
-    (effects (font (size 1.27 1.27)) (justify left bottom))
-  )
   (label "SCL" (at 127.635 55.88 0)
     (effects (font (size 1.27 1.27)) (justify left bottom))
@@
     (effects (font (size 1.27 1.27)) (justify left bottom))
   )
+  (label "GP4_DONE" (at 165.1 52.07 180)
+    (effects (font (size 1.27 1.27)) (justify right bottom))
+  )
   (label "SCL" (at 99.06 76.2 0)
     (effects (font (size 1.27 1.27)) (justify left bottom))
@@
     (effects (font (size 1.27 1.27)) (justify left bottom))
   )
-  (label "GP5_DONE" (at 165.1 52.07 180)
-    (effects (font (size 1.27 1.27)) (justify right bottom))
-  )
-  (label "GP4_CLKOUT" (at 127.635 120.015 0)
+  (label "GP4_DONE" (at 127.635 120.015 0)
     (effects (font (size 1.27 1.27)) (justify left bottom))
   )
@@
   )
   (label "CLKOUT" (at 127 81.28 0)
+    (effects (font (size 1.27 1.27)) (justify left bottom))
+  )
+  (label "GP5_CLKOUT" (at 127 90.17 0)
     (effects (font (size 1.27 1.27)) (justify left bottom))
   )
@@
   )
   (symbol (lib_id "Connector_Generic:Conn_01x02") (at 173.99 104.14 0) (unit 1)
-    (in_bom yes) (on_board yes) (fields_autoplaced)
+    (in_bom no) (on_board yes) (fields_autoplaced)
     (property "Reference" "J1" (id 0) (at 176.022 104.5753 0)
       (effects (font (size 1.27 1.27)) (justify left))
@@
   )
   (symbol (lib_id "Connector_Generic:Conn_01x13") (at 93.98 123.19 0) (unit 1)
-    (in_bom yes) (on_board yes)
+    (in_bom no) (on_board yes)
     (property "Reference" "J3" (id 0) (at 92.71 101.6 0)
       (effects (font (size 1.27 1.27)) (justify left))
@@
   )
   (symbol (lib_id "user:SW_Push_SLIM") (at 169.545 74.93 0) (unit 1)
-    (in_bom yes) (on_board yes) (fields_autoplaced)
+    (in_bom no) (on_board yes) (fields_autoplaced)
     (property "Reference" "SW1" (id 0) (at 169.545 68.3092 0))
     (property "Value" "SW_Push_SLIM" (id 1) (at 169.545 70.8461 0))
@@
   )
   (symbol (lib_id "Connector_Generic:Conn_01x02") (at 173.99 113.03 0) (unit 1)
-    (in_bom yes) (on_board yes) (fields_autoplaced)
+    (in_bom no) (on_board yes) (fields_autoplaced)
     (property "Reference" "J4" (id 0) (at 176.022 113.4653 0)
       (effects (font (size 1.27 1.27)) (justify left))
@@
   )
   (symbol (lib_id "Connector_Generic:Conn_01x13") (at 118.745 122.555 0) (mirror y) (unit 1)
-    (in_bom yes) (on_board yes)
+    (in_bom no) (on_board yes)
     (property "Reference" "J2" (id 0) (at 120.65 101.6 0)
       (effects (font (size 1.27 1.27)) (justify left))
